Commit message: remove gripper

File: dual_arm_scene_description/urdf/base_scene.urdf.xacro (robot description, xacro)
@@ -77,7 +77,7 @@
   <!-- Spawn and attach robotiq grippers -->
   <xacro:include filename="$(find dual_arm_scene_description)/urdf/components/dual_arm_end_effector_2F-140.urdf.xacro" />
-  <xacro:dual_arm_end_effector prefix="a_bot_" use_soft_wrist="false" parent = "a_bot_ee_link" />
+  <xacro:dual_arm_end_effector prefix="a_bot_" parent = "a_bot_ee_link" />
   <xacro:include filename="$(find dual_arm_scene_description)/urdf/components/dual_arm_end_effector.urdf.xacro" />
-  <xacro:dual_arm_end_effector prefix="b_bot_" use_soft_wrist="false" parent = "b_bot_ee_link" />
+  <xacro:dual_arm_end_effector prefix="b_bot_" parent = "b_bot_ee_link" />
   <!-- The "world" link definition should be removed, but apparently it is necessary for Gazebo -->
   <link name="world" />

File: dual_arm_scene_description/urdf/components/dual_arm_end_effector.urdf.xacro (robot description, xacro)
@@ -3,9 +3,9 @@
 <!-- The position of the TF frame has not been measured at all and needs to be calibrated. -->
 <robot name="robotiq_85_gripper_test" xmlns:xacro="http://www.ros.org/wiki/xacro">
-  <xacro:macro name="dual_arm_end_effector" params="prefix use_soft_wrist:=false parent">
-    <xacro:include filename="$(find robotiq_description)/urdf/robotiq_85_gripper.urdf.xacro"/>
-    <xacro:robotiq_85_gripper prefix="${prefix}" parent="${parent}">
-        <origin rpy="0.0 0.0 0.0" xyz="0.01 0 0"/> <!-- This 0.01 offset is the Robotiq/UR coupling -->
-    </xacro:robotiq_85_gripper>
+  <xacro:macro name="dual_arm_end_effector" params="prefix parent">
+    <!-- <xacro:include filename="$(find robotiq_description)/urdf/robotiq_85_gripper.urdf.xacro"/> -->
+    <!-- <xacro:robotiq_85_gripper prefix="${prefix}" parent="${parent}">
+        <origin rpy="0.0 0.0 0.0" xyz="0.01 0 0"/>
+    </xacro:robotiq_85_gripper> -->
     <link name="${prefix}_coupling">
       <visual>
@@ -32,5 +32,5 @@
     <!-- Add an additional link to plan with. Oriented like the UR ee_link frame. -->
     <joint name="${prefix}robotiq_85_tip_link_joint" type="fixed">
-      <parent link="${prefix}robotiq_85_base_link"/>
+      <parent link="${parent}"/>
       <child link="${prefix}robotiq_85_tip_link"/>
       <origin rpy="0 0 0" xyz=".163 0 0"/>

File: dual_arm_scene_description/urdf/components/dual_arm_end_effector_2F-140.urdf.xacro (robot description, xacro)
@@ -3,12 +3,12 @@
      instead of a 2F-85 gripper. The tip link is set to the . -->
 <robot name="robotiq_85_gripper_test" xmlns:xacro="http://www.ros.org/wiki/xacro">
-  <xacro:macro name="dual_arm_end_effector" params="prefix use_soft_wrist:=false parent">
-    <xacro:include filename="$(find robotiq_description)/urdf/robotiq_140_gripper.urdf.xacro"/>
-    <xacro:robotiq_140_gripper prefix="${prefix}" parent="${parent}">
+  <xacro:macro name="dual_arm_end_effector" params="prefix parent">
+    <!-- <xacro:include filename="$(find robotiq_description)/urdf/robotiq_140_gripper.urdf.xacro"/> -->
+    <!-- <xacro:robotiq_140_gripper prefix="${prefix}" parent="${parent}">
         <origin rpy="0.0 0.0 0.0" xyz="0 0 0"/>
-    </xacro:robotiq_140_gripper>
+    </xacro:robotiq_140_gripper> -->
     <!-- Add an additional link to plan with. Oriented like the UR ee_link frame. -->
     <joint name="${prefix}robotiq_85_tip_link_joint" type="fixed">
-      <parent link="${prefix}robotiq_140_base_link"/>
+      <parent link="${parent}"/>
       <child link="${prefix}robotiq_85_tip_link"/>
       <origin rpy="0.0 0.0 0.0" xyz="${.163+.083} 0.0 0.0"/>
